File: hardware/Daneben_Prototype_Carrier_Board/Daneben_Prototype_Carrier_Board.kicad_sch (KiCad schematic)
At the start: 23 parts

Commit message: fix(hardware): Update schematic pin alignment script and prototype BOM
Connections:
- net D_NEG: no longer names the net of J_USBC.3 (Pin_3)
- net D_POS: no longer names the net of J_USBC.4 (Pin_4)
- no-connect marks 0 -> 2
Changed lines of the file:
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@@
 		(effects (font (size 1.27 1.27)))
 	)
-	(wire (pts (xy 35.56 63.50) (xy 45.72 63.50))
-		(stroke (width 0) (type default))
-	)
-	(label "D_NEG"
-		(at 35.56 63.50 180)
-		(effects (font (size 1.27 1.27)))
-	)
-	(wire (pts (xy 35.56 66.04) (xy 45.72 66.04))
-		(stroke (width 0) (type default))
-	)
-	(label "D_POS"
-		(at 35.56 66.04 180)
-		(effects (font (size 1.27 1.27)))
+	(no_connect
+		(at 45.72 63.50)
+	)
+	(no_connect
+		(at 45.72 66.04)
 	)
 	(wire (pts (xy 35.56 68.58) (xy 45.72 68.58))
@@
 		(effects (font (size 1.27 1.27)))
 	)
-	(wire (pts (xy 125.73 50.80) (xy 129.54 50.80))
-		(stroke (width 0) (type default))
-	)
 	(symbol
 		(lib_id "Device:LED")
-		(at 133.35 50.80 180)
-		(unit 1)
-		(in_bom yes) (on_board yes)
-		(property "Reference" "LED_PWR" (at 133.35 46.30 0) (effects (font (size 1.27 1.27))))
-		(property "Value" "GREEN (PWR)" (at 133.35 55.30 0) (effects (font (size 1.27 1.27))))
-		(property "Footprint" "LED_THT:LED_D3.0mm" (at 133.35 50.80 0) (effects (font (size 1.27 1.27)) (hide yes)))
-	)
-	(wire (pts (xy 137.16 50.80) (xy 142.24 50.80))
+		(at 129.54 50.80 180)
+		(unit 1)
+		(in_bom yes) (on_board yes)
+		(property "Reference" "LED_PWR" (at 129.54 46.30 0) (effects (font (size 1.27 1.27))))
+		(property "Value" "GREEN (PWR)" (at 129.54 55.30 0) (effects (font (size 1.27 1.27))))
+		(property "Footprint" "LED_THT:LED_D3.0mm" (at 129.54 50.80 0) (effects (font (size 1.27 1.27)) (hide yes)))
+	)
+	(wire (pts (xy 133.35 50.80) (xy 142.24 50.80))
 		(stroke (width 0) (type default))
 	)
@@
 		(effects (font (size 1.27 1.27)))
 	)
-	(wire (pts (xy 240.03 185.42) (xy 243.84 185.42))
-		(stroke (width 0) (type default))
-	)
 	(symbol
 		(lib_id "Device:LED")
-		(at 247.65 185.42 180)
-		(unit 1)
-		(in_bom yes) (on_board yes)
-		(property "Reference" "LED_CAL_OUT" (at 247.65 180.92 0) (effects (font (size 1.27 1.27))))
-		(property "Value" "BLUE (OUT_STAT)" (at 247.65 189.92 0) (effects (font (size 1.27 1.27))))
-		(property "Footprint" "LED_THT:LED_D3.0mm" (at 247.65 185.42 0) (effects (font (size 1.27 1.27)) (hide yes)))
-	)
-	(wire (pts (xy 251.46 185.42) (xy 259.08 185.42))
+		(at 243.84 185.42 180)
+		(unit 1)
+		(in_bom yes) (on_board yes)
+		(property "Reference" "LED_CAL_OUT" (at 243.84 180.92 0) (effects (font (size 1.27 1.27))))
+		(property "Value" "BLUE (OUT_STAT)" (at 243.84 189.92 0) (effects (font (size 1.27 1.27))))
+		(property "Footprint" "LED_THT:LED_D3.0mm" (at 243.84 185.42 0) (effects (font (size 1.27 1.27)) (hide yes)))
+	)
+	(wire (pts (xy 247.65 185.42) (xy 259.08 185.42))
 		(stroke (width 0) (type default))
 	)
@@
 		(effects (font (size 1.27 1.27)))
 	)
-	(wire (pts (xy 240.03 220.98) (xy 243.84 220.98))
-		(stroke (width 0) (type default))
-	)
 	(symbol
 		(lib_id "Device:LED")
-		(at 247.65 220.98 180)
-		(unit 1)
-		(in_bom yes) (on_board yes)
-		(property "Reference" "LED_CAL_IN" (at 247.65 216.48 0) (effects (font (size 1.27 1.27))))
-		(property "Value" "AMBER (IN_STAT)" (at 247.65 225.48 0) (effects (font (size 1.27 1.27))))
-		(property "Footprint" "LED_THT:LED_D3.0mm" (at 247.65 220.98 0) (effects (font (size 1.27 1.27)) (hide yes)))
-	)
-	(wire (pts (xy 251.46 220.98) (xy 259.08 220.98))
-		(stroke (width 0) (type default))
-	)
+		(at 243.84 220.98 180)
+		(unit 1)
+		(in_bom yes) (on_board yes)
+		(property "Reference" "LED_CAL_IN" (at 243.84 216.48 0) (effects (font (size 1.27 1.27))))
+		(property "Value" "AMBER (IN_STAT)" (at 243.84 225.48 0) (effects (font (size 1.27 1.27))))
+		(property "Footprint" "LED_THT:LED_D3.0mm" (at 243.84 220.98 0) (effects (font (size 1.27 1.27)) (hide yes)))
+	)
+	(wire (pts (xy 247.65 220.98) (xy 259.08 220.98))
+		(stroke (width 0) (type default))
+	)
